File: Progenitor-Tenkey.kicad_pcb (KiCad board)
At the start: 2 copper layers, 359.6 x 114.3 mm, 208 parts, among them SW1 SW_Push, U1 ATmega32U4-AU, Y1 16MHz

Commit message: Small Tweaks
Parts:
- USB1: value Molex-0548190519 -> Molex-0548190589
- moved USB1 1.40 mm to (360.0, 232.8)
Connections:
- USB1 pad 6: Net-(USB1-Pad6) -> GND
Routing:
- net D-: track 6.82 -> 8.32 mm
- net D+: track 6.82 -> 8.32 mm
- net GND: track 171.7 -> 173.2 mm
- net VCC: track 12.4 -> 13.6 mm
- net Net-(R3-Pad2): track 32.8 -> 33.4 mm
- added copper zone on B.Cu, net GND
Other:
- outline, holes or cut-outs redrawn

Commit message: Aesthetic Tweak
Other:
- board text added: "PROGENITOR Rev.1"
- board text added: "Taylor Simpson"
Changed lines of the file:
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@@
   (general
     (thickness 1.6)
-    (drawings 10)
+    (drawings 12)
     (tracks 1435)
     (zones 0)
@@
     )
   )
+  (gr_text "Taylor Simpson" (at 369.09375 312.7375) (layer F.SilkS)
+    (effects (font (size 1 1) (thickness 0.15)))
+  )
+  (gr_text "PROGENITOR Rev.1" (at 372.26875 311.15) (layer F.SilkS)
+    (effects (font (size 1.27 1.27) (thickness 0.254)))
+  )
   (gr_line (start 356.39375 230.98125) (end 364.33125 230.98125) (layer Edge.Cuts) (width 0.05))
   (gr_line (start 356.39375 230.98125) (end 82.55 230.98125) (layer Edge.Cuts) (width 0.05))
@@
       )
     )
+  )
+  (zone (net 1) (net_name GND) (layer B.Cu) (hatch edge 0.508)
+    (connect_pads (clearance 0.508))
+    (min_thickness 0.254)
+    (fill yes (arc_segments 32) (thermal_gap 0.508) (thermal_bridge_width 0.508))
+    (polygon
+      (pts
+        (xy 376.682 326.517) (xy 368.554 318.389) (xy 368.554 311.531) (xy 372.618 307.467) (xy 395.732 307.467)
+      )
+    )
+  )
+  (zone (net 0) (net_name "") (layer B.SilkS) (hatch edge 0.508)
+    (connect_pads (clearance 0.508))
+    (min_thickness 0.254)
+    (fill yes (arc_segments 32) (thermal_gap 0.508) (thermal_bridge_width 0.508))
+    (polygon
+      (pts
+        (xy 156.36875 345.28125) (xy 99.21875 345.28125) (xy 213.51875 230.98125) (xy 270.66875 230.98125)
+      )
+    )
+  )
+  (zone (net 0) (net_name "") (layer B.SilkS) (hatch edge 0.508)
+    (connect_pads (clearance 0.508))
+    (min_thickness 0.254)
+    (fill yes (arc_segments 32) (thermal_gap 0.508) (thermal_bridge_width 0.508))
+    (polygon
+      (pts
+        (xy 225.425 345.28125) (xy 168.275 345.28125) (xy 282.575 230.98125) (xy 339.725 230.98125)
+      )
+    )
