File: Progenitor-Tenkey.kicad_pcb (KiCad board)
At the start: 2 copper layers, 359.6 x 114.3 mm, 208 parts, among them SW1 SW_Push, U1 ATmega32U4-AU, Y1 16MHz

Commit message: More tweaks, regenerated Gerber
Parts:
- R1, R2: value R_Small -> 22
- moved C1 162.1 mm to (324.7, 158.0)
- moved C3 162.1 mm to (329.6, 156.5)
- moved C5 162.1 mm to (317.9, 176.8)
- moved C6 162.1 mm to (313.6, 160.3)
- moved D10 162.1 mm to (67.7, 181.2)
- moved D15 162.1 mm to (86.7, 181.2)
- moved D21 162.1 mm to (105.8, 181.2)
- moved D42 162.1 mm to (174.8, 181.2)
- moved D58 162.1 mm to (246.3, 181.2)
- moved D6 162.1 mm to (48.6, 181.2)
- moved D64 162.1 mm to (272.4, 181.2)
- moved D76 162.1 mm to (301.0, 181.2)
- moved D85 162.1 mm to (351.0, 181.2)
- moved D91 162.1 mm to (370.1, 181.2)
- moved D96 162.1 mm to (389.1, 181.2)
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Routing:
- net GND: track 173.2 -> 169.8 mm, vias 0 -> 4
- net +5V: track 125.5 -> 125.1 mm, vias 4 -> 0
