File: Project Files/Progenitor-TenkeyR2.kicad_pcb (KiCad board)
At the start: 2 copper layers, 362 x 116.7 mm, 208 parts, among them SW1 SW_Push, U1 ATmega32U4-AU, Y1 16MHz

Commit message: Board Rev.2
Parts:
- moved C1 4.56 mm to (324.7, 158.0), turned to 315 degrees
- moved C7 3.48 mm to (311.3, 170.3), turned to 315 degrees
- moved C2 2.50 mm to (335.2, 162.1)
- moved C3 2.50 mm to (329.6, 156.5)
- moved Y1 2.50 mm to (332.3, 159.3)
- moved C5 2.42 mm to (317.9, 176.8), turned to 135 degrees
- moved C4 2.39 mm to (329.3, 170.1), turned to 45 degrees
- moved R3 1.91 mm to (322.2, 156.5), turned to 225 degrees
- moved C6 1.63 mm to (313.6, 160.3), turned to 225 degrees
- moved R4 1.15 mm to (321.4, 179.1), turned to 45 degrees
Connections:
- U1 pad 1: ROW04 -> COL08
- U1 pad 11: ROW03 -> COL14
- U1 pad 12: Net-(U1-Pad12) -> ROW03
- U1 pad 18: ROW05 -> COL00
- U1 pad 19: COL14 -> COL01
- U1 pad 20: COL15 -> Net-(U1-Pad20)
- U1 pad 21: COL16 -> COL02
- U1 pad 22: COL17 -> COL03
- U1 pad 25: COL00 -> COL04
- U1 pad 26: COL01 -> COL05
- U1 pad 27: COL02 -> COL06
- U1 pad 28: COL03 -> COL07
- U1 pad 29: COL04 -> COL15
- U1 pad 30: COL05 -> COL16
- U1 pad 31: COL06 -> COL17
- U1 pad 32: COL07 -> ROW05
- U1 pad 36: COL08 -> COL09
- U1 pad 37: COL09 -> COL10
- U1 pad 38: COL10 -> COL11
- U1 pad 39: COL11 -> COL12
- U1 pad 40: COL12 -> COL13
- U1 pad 41: COL13 -> ROW04
Routing:
- net ROW00: track 365.4 -> 592.8 mm, vias 18 -> 2
- net ROW01: track 365.4 -> 573.9 mm, vias 18 -> 2
- net ROW04: track 280.2 -> 470.7 mm, vias 15 -> 3
- net ROW02: track 360.6 -> 548.3 mm, vias 18 -> 2
- net ROW03: track 359.2 -> 518.9 mm, vias 17 -> 2
- net GND: track 17.2 -> 169.8 mm, vias 0 -> 4
- net ROW05: track 357.7 -> 441.7 mm, vias 12 -> 2
- net COL01: track 398.9 -> 475.4 mm, vias 0 -> 1
- net COL00: track 416.2 -> 489.6 mm, vias 0 -> 1
- net COL14: track 131.0 -> 82.3 mm, vias 0 -> 1
- net COL02: track 389.2 -> 412.8 mm, vias 0 -> 3
- net COL15: track 141.6 -> 119.0 mm
- net +5V: track 142.7 -> 125.1 mm, vias 7 -> 0
- net COL05: track 319.3 -> 334.7 mm, vias 0 -> 3
- net COL07: track 288.0 -> 303.4 mm, vias 0 -> 3
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- added copper zone on B.Cu, net GND
Other:
- board size 362 x 116.7 mm -> 359.6 x 114.3 mm
