File: Project Files/Progenitor-Tenkey.kicad_pcb (KiCad board)
At the start: 2 copper layers, 359.6 x 114.3 mm, 208 parts, among them SW1 SW_Push, U1 ATmega32U4-AU, Y1 16MHz

Commit message: Board Rev.2
Parts:
- moved C1 4.56 mm to (320.3, 159.0), turned to 0 degrees
- moved C7 3.48 mm to (308.8, 167.9), turned to 270 degrees
- moved C2 2.50 mm to (332.7, 161.4)
- moved C3 2.50 mm to (327.2, 155.8)
- moved Y1 2.50 mm to (329.9, 158.7)
- moved C5 2.42 mm to (320.3, 176.7), turned to 180 degrees
- moved C4 2.39 mm to (329.1, 167.8), turned to 90 degrees
- moved R3 1.91 mm to (320.3, 156.6), turned to 0 degrees
- moved C6 1.63 mm to (312.5, 159.0), turned to 90 degrees
- moved R4 1.15 mm to (320.3, 178.9), turned to 0 degrees
Connections:
- U1 pad 1: COL08 -> ROW05
- U1 pad 11: COL14 -> ROW03
- U1 pad 12: ROW03 -> Net-(U1-Pad12)
- U1 pad 18: COL00 -> ROW04
- U1 pad 19: COL01 -> COL14
- U1 pad 20: Net-(U1-Pad20) -> COL15
- U1 pad 21: COL02 -> COL16
- U1 pad 22: COL03 -> COL17
- U1 pad 25: COL04 -> COL00
- U1 pad 26: COL05 -> COL01
- U1 pad 27: COL06 -> COL02
- U1 pad 28: COL07 -> COL03
- U1 pad 29: COL15 -> COL04
- U1 pad 30: COL16 -> COL05
- U1 pad 31: COL17 -> COL06
- U1 pad 32: ROW05 -> COL07
- U1 pad 36: COL09 -> COL08
- U1 pad 37: COL10 -> COL09
- U1 pad 38: COL11 -> COL10
- U1 pad 39: COL12 -> COL11
- U1 pad 40: COL13 -> COL12
- U1 pad 41: ROW04 -> COL13
Routing:
- net ROW01: track 573.9 -> 420.7 mm, vias 2 -> 19
- net ROW00: track 592.8 -> 440.4 mm, vias 2 -> 19
- net ROW02: track 548.3 -> 396.2 mm, vias 2 -> 19
- net ROW03: track 518.9 -> 375.1 mm, vias 2 -> 18
- net GND: track 169.8 -> 31.3 mm, vias 4 -> 0
- net ROW04: track 470.7 -> 357.2 mm, vias 3 -> 15
- net COL01: track 475.4 -> 398.9 mm, vias 1 -> 0
- net COL00: track 489.6 -> 416.2 mm, vias 1 -> 0
- net ROW05: track 441.7 -> 381.3 mm, vias 2 -> 14
- net COL14: track 82.3 -> 131.0 mm, vias 1 -> 0
- net COL02: track 412.8 -> 389.2 mm, vias 3 -> 0
- net COL15: track 119.0 -> 141.6 mm
- net +5V: track 125.1 -> 142.7 mm, vias 0 -> 7
- net COL05: track 334.7 -> 319.3 mm, vias 3 -> 0
- net COL07: track 303.4 -> 288.0 mm, vias 3 -> 0
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Other:
- board size 359.6 x 114.3 mm -> 362 x 116.7 mm

Commit message: Fixed Bugs
Other:
- board size 362 x 116.7 mm -> 361.9 x 117.5 mm
Changed lines of the file:
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@@
   (general
     (thickness 1.6)
-    (drawings 10)
+    (drawings 12)
     (tracks 1392)
     (zones 0)
@@
     )
   )
-  (gr_line (start 30.95625 192.0875) (end 391.31875 192.0875) (layer Edge.Cuts) (width 0.05))
+  (gr_line (start 392.1125 192.0875) (end 392.1125 191.29375) (layer Edge.Cuts) (width 0.05))
+  (gr_line (start 30.1625 192.0875) (end 30.1625 191.29375) (layer Edge.Cuts) (width 0.05))
+  (gr_line (start 30.95625 192.88125) (end 391.31875 192.88125) (layer Edge.Cuts) (width 0.05))
   (gr_line (start 30.1625 76.2) (end 30.1625 191.29375) (layer Edge.Cuts) (width 0.05))
   (gr_line (start 391.31875 75.40625) (end 30.95625 75.40625) (layer Edge.Cuts) (width 0.05))
   (gr_line (start 392.1125 191.29375) (end 392.1125 76.2) (layer Edge.Cuts) (width 0.05))
-  (gr_arc (start 391.31875 191.29375) (end 391.31875 192.0875) (angle -90) (layer Edge.Cuts) (width 0.05))
+  (gr_arc (start 391.31875 192.0875) (end 391.31875 192.88125) (angle -90) (layer Edge.Cuts) (width 0.05))
   (gr_arc (start 391.31875 76.2) (end 392.1125 76.2) (angle -90) (layer Edge.Cuts) (width 0.05))
   (gr_arc (start 30.95625 76.2) (end 30.95625 75.40625) (angle -90) (layer Edge.Cuts) (width 0.05))
-  (gr_arc (start 30.95625 191.29375) (end 30.1625 191.29375) (angle -90) (layer Edge.Cuts) (width 0.05))
+  (gr_arc (start 30.95625 192.0875) (end 30.1625 192.0875) (angle -90) (layer Edge.Cuts) (width 0.05))
   (gr_text "Taylor Simpson" (at 320.07175 158.1785) (layer F.SilkS)
     (effects (font (size 1 1) (thickness 0.15)))

Commit message: Fixed Errors
Parts:
- removed MX-RCT1: MX-NoLED, MX_Only:MXOnly-1.5U-NoLED
- moved C1 2.03 mm to (320.3, 157.0)
- moved C4 1.78 mm to (330.8, 167.8)
- moved C5 1.66 mm to (320.4, 178.3)
- moved R3 1.65 mm to (320.3, 154.9)
- moved R4 1.53 mm to (320.4, 180.5)
Routing:
- net +5V: track 142.7 -> 148.1 mm
- net GND: track 31.3 -> 35.5 mm
- net COL00: track 416.2 -> 418.4 mm
- net COL01: track 398.9 -> 401.0 mm
- net COL06: track 298.8 -> 300.7 mm
- net COL03: track 368.7 -> 370.5 mm
- net COL02: track 389.2 -> 391.0 mm
- net COL04: track 339.8 -> 341.6 mm
- net COL05: track 319.3 -> 320.9 mm
- net COL16: track 152.8 -> 154.2 mm
- net COL15: track 141.6 -> 142.9 mm
- net COL07: track 288.0 -> 289.3 mm
- net COL17: track 171.0 -> 172.3 mm
- net Net-(R4-Pad2): track 7.03 -> 8.14 mm
